Commit message: phase 1 working

File: install/f1tenth_gazebo/share/f1tenth_gazebo/urdf/racecar_blue.xacro (robot description, xacro)
@@ -34,5 +34,5 @@
       <material name="black" />
     </visual>
-    <collision>robot
+    <collision>
       <xacro:left_wheels_collision_geometry />
     </collision>
@@ -77,10 +77,11 @@
     </visual>
   </link>
-  <joint name="left_steering_hinge_joint" type="fixed">
-    <origin xyz="0.325 0.1 0" rpy="0 1.5708 0" />
+  <joint name="left_steering_hinge_joint" type="revolute">
+    <origin xyz="0.325 0.1 0" rpy="0 0 0" />
     <parent link="chassis" />
     <child link="left_steering_hinge" />
-    <axis xyz="-1 0 0" />
-    <limit lower="-1.0" upper="1.0" effort="10" velocity="100" />
+    <axis xyz="0 0 1" />
+    <limit lower="-0.5" upper="0.5" effort="10" velocity="1.0" />
+    <dynamics damping="0.5" friction="0.0" />
   </joint>
   <xacro:steering_hinge_transmission name="left_steering_hinge" />
@@ -95,10 +96,11 @@
     </visual>
   </link>
-  <joint name="right_steering_hinge_joint" type="fixed">
-    <origin xyz="0.325 -0.1 0" rpy="0 1.5708 0" />
+  <joint name="right_steering_hinge_joint" type="revolute">
+    <origin xyz="0.325 -0.1 0" rpy="0 0 0" />
     <parent link="chassis" />
     <child link="right_steering_hinge" />
-    <axis xyz="-1 0 0" />
-    <limit lower="-1.0" upper="1.0" effort="10" velocity="100" />
+    <axis xyz="0 0 1" />
+    <limit lower="-0.5" upper="0.5" effort="10" velocity="1.0" />
+    <dynamics damping="0.5" friction="0.0" />
   </joint>
   <xacro:steering_hinge_transmission name="right_steering_hinge" />
@@ -124,5 +126,5 @@
   </joint>
   <xacro:wheel_transmission name="left_front_wheel" />
-  <!-- Add the left front wheel with its joints and tranmissions -->
+  <!-- Add the right front wheel with its joints and tranmissions -->
   <link name="right_front_wheel">
     <inertial>
@@ -227,4 +229,5 @@
   </joint>
   <!-- Add the remaining xacros -->
+  <xacro:property name="lidar_topic" value="blue_scan" />
   <xacro:include filename="$(find f1tenth_gazebo)/urdf/racecar.gazebo" />
   <xacro:include filename="$(find f1tenth_gazebo)/urdf/materials.xacro" />

File: install/f1tenth_gazebo/share/f1tenth_gazebo/urdf/racecar_green.xacro (robot description, xacro)
@@ -34,5 +34,5 @@
       <material name="black" />
     </visual>
-    <collision>robot
+    <collision>
       <xacro:left_wheels_collision_geometry />
     </collision>
@@ -77,10 +77,11 @@
     </visual>
   </link>
-  <joint name="left_steering_hinge_joint" type="fixed">
-    <origin xyz="0.325 0.1 0" rpy="0 1.5708 0" />
+  <joint name="left_steering_hinge_joint" type="revolute">
+    <origin xyz="0.325 0.1 0" rpy="0 0 0" />
     <parent link="chassis" />
     <child link="left_steering_hinge" />
-    <axis xyz="-1 0 0" />
-    <limit lower="-1.0" upper="1.0" effort="10" velocity="100" />
+    <axis xyz="0 0 1" />
+    <limit lower="-0.5" upper="0.5" effort="10" velocity="1.0" />
+    <dynamics damping="0.5" friction="0.0" />
   </joint>
   <xacro:steering_hinge_transmission name="left_steering_hinge" />
@@ -95,10 +96,11 @@
     </visual>
   </link>
-  <joint name="right_steering_hinge_joint" type="fixed">
-    <origin xyz="0.325 -0.1 0" rpy="0 1.5708 0" />
+  <joint name="right_steering_hinge_joint" type="revolute">
+    <origin xyz="0.325 -0.1 0" rpy="0 0 0" />
     <parent link="chassis" />
     <child link="right_steering_hinge" />
-    <axis xyz="-1 0 0" />
-    <limit lower="-1.0" upper="1.0" effort="10" velocity="100" />
+    <axis xyz="0 0 1" />
+    <limit lower="-0.5" upper="0.5" effort="10" velocity="1.0" />
+    <dynamics damping="0.5" friction="0.0" />
   </joint>
   <xacro:steering_hinge_transmission name="right_steering_hinge" />
@@ -124,5 +126,5 @@
   </joint>
   <xacro:wheel_transmission name="left_front_wheel" />
-  <!-- Add the left front wheel with its joints and tranmissions -->
+  <!-- Add the right front wheel with its joints and tranmissions -->
   <link name="right_front_wheel">
     <inertial>
@@ -227,4 +229,5 @@
   </joint>
   <!-- Add the remaining xacros -->
+  <xacro:property name="lidar_topic" value="green_scan" />
   <xacro:include filename="$(find f1tenth_gazebo)/urdf/racecar.gazebo" />
   <xacro:include filename="$(find f1tenth_gazebo)/urdf/materials.xacro" />

File: install/f1tenth_gazebo/share/f1tenth_gazebo/urdf/racecar_red.xacro (robot description, xacro)
@@ -34,5 +34,5 @@
       <material name="black" />
     </visual>
-    <collision>robot
+    <collision>
       <xacro:left_wheels_collision_geometry />
     </collision>
@@ -77,10 +77,11 @@
     </visual>
   </link>
-  <joint name="left_steering_hinge_joint" type="fixed">
-    <origin xyz="0.325 0.1 0" rpy="0 1.5708 0" />
+  <joint name="left_steering_hinge_joint" type="revolute">
+    <origin xyz="0.325 0.1 0" rpy="0 0 0" />
     <parent link="chassis" />
     <child link="left_steering_hinge" />
-    <axis xyz="-1 0 0" />
-    <limit lower="-1.0" upper="1.0" effort="10" velocity="100" />
+    <axis xyz="0 0 1" />
+    <limit lower="-0.5" upper="0.5" effort="10" velocity="1.0" />
+    <dynamics damping="0.5" friction="0.0" />
   </joint>
   <xacro:steering_hinge_transmission name="left_steering_hinge" />
@@ -95,10 +96,11 @@
     </visual>
   </link>
-  <joint name="right_steering_hinge_joint" type="fixed">
-    <origin xyz="0.325 -0.1 0" rpy="0 1.5708 0" />
+  <joint name="right_steering_hinge_joint" type="revolute">
+    <origin xyz="0.325 -0.1 0" rpy="0 0 0" />
     <parent link="chassis" />
     <child link="right_steering_hinge" />
-    <axis xyz="-1 0 0" />
-    <limit lower="-1.0" upper="1.0" effort="10" velocity="100" />
+    <axis xyz="0 0 1" />
+    <limit lower="-0.5" upper="0.5" effort="10" velocity="1.0" />
+    <dynamics damping="0.5" friction="0.0" />
   </joint>
   <xacro:steering_hinge_transmission name="right_steering_hinge" />
@@ -227,4 +229,5 @@
   </joint>
   <!-- Add the remaining xacros -->
+  <xacro:property name="lidar_topic" value="red_scan" />
   <xacro:include filename="$(find f1tenth_gazebo)/urdf/racecar.gazebo" />
   <xacro:include filename="$(find f1tenth_gazebo)/urdf/materials.xacro" />
